File: ChargingBoard/ChargingBoard/ChargingBoard.kicad_pcb (KiCad board)
At the start: 4 copper layers, 125 x 50 mm, 145 parts, among them J1 Conn_02x03_Odd_Even, J17 Micro_SD_Card, J2 Screw_Terminal_01x02, J3 Screw_Terminal_01x02, J4 Screw_Terminal_01x02, J5 Screw_Terminal_01x02, J6 Conn_01x03_Pin, J7 Screw_Terminal_01x02, Q1 FQP27P06, Q10 FDC658AP, Q12 IRLZ44N, Q16 IRLZ44N, Q2 FQP27P06, Q3 FQP27P06, Q4 IRLZ44N, Q5 FQP27P06, Q6 FQP27P06, Q7 FQP27P06, Q8 IRLZ44N, Q9 FDC658AP, U1 LTC4011CFE, U10 FDS6975, U11 FDS6975, U2 LTC4011CFE, U3 LP2985-3.3, U4 LTC4011CFE, U5 LTC4011CFE, U6 ATmega328P-A, U7 INA260, U8 INA260, U9 CD4050BPWR, Y1 16MHz

Commit message: Arrangement Begins
Parts:
- BT1, BT2, BT3, BT4: footprint TerminalBlock_Phoenix:TerminalBlock_Phoenix_MKDS-1,5-2-5.08_1x02_P5.08mm_Horizontal -> TerminalBlock_Phoenix:TerminalBlock_Phoenix_MPT-0,5-2-2.54_1x02_P2.54mm_Horizontal
- D10, D5: footprint Diode_SMD:D_SMA-SMB_Universal_Handsoldering -> Diode_SMD:D_SMA_Handsoldering
- D15, D20: footprint Diode_SMD:D_SMA-SMB_Universal_Handsoldering -> Diode_SMD:D_SOD-323_HandSoldering
- J2, J3, J4, J5, J7: footprint TerminalBlock_Phoenix:TerminalBlock_Phoenix_MKDS-1,5-2-5.08_1x02_P5.08mm_Horizontal -> TerminalBlock_Phoenix:TerminalBlock_Phoenix_MKDS-1-2-3.81_1x02_P3.81mm_Horizontal
- moved J17 194.2 mm to (238.3, 122.1)
- moved U9 183.6 mm to (238.0, 108.9), turned to -90 degrees
- moved R1 181.2 mm to (248.5, 24.6)
- moved R2 181.2 mm to (248.5, 27.1)
- moved R3 181.2 mm to (248.5, 29.7)
- moved R4 181.2 mm to (248.5, 32.2)
- moved J1 173.6 mm to (241.0, 102.3), turned to -90 degrees
- moved R11 168.7 mm to (246.3, 42.9), turned to 90 degrees
- moved R8 167.4 mm to (245.1, 35.7)
- moved Q9 164.9 mm to (41.2, 177.9)
- moved J6 159.3 mm to (233.1, 81.5), turned to 90 degrees
- moved C1 158.9 mm to (228.8, 33.9)
- moved C2 158.9 mm to (228.8, 36.4)
- moved C3 158.9 mm to (228.8, 38.9)
- moved C23 158.1 mm to (230.0, 107.4), turned to 180 degrees
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Routing:
- net /RESET: track 0.00 -> 16.1 mm, vias 0 -> 1
- net /SCK: track 0.00 -> 13.4 mm
- net Net-(U6-XTAL2/PB7): track 0.00 -> 8.34 mm
- net Net-(U6-XTAL1/PB6): track 0.00 -> 8.19 mm
- net /MISO: track 0.00 -> 6.73 mm
- net /MOSI: track 0.00 -> 4.26 mm
- net GND: track 0.00 -> 3.07 mm, vias 0 -> 3
- net /TX: track 0.00 -> 2.92 mm
- net /RX: track 0.00 -> 2.84 mm
- net Net-(U1-TIMER): track 0.00 -> 2.31 mm
- net Net-(U6-PD1): track 0.00 -> 2.19 mm
- net Net-(U6-PD0): track 0.00 -> 2.19 mm
- net +3V3: track 0.00 -> 2.06 mm
- net +5V: track 0.00 -> 1.84 mm
- added copper zone on In1.Cu, net GND
Other:
- board size 125 x 50 mm -> 125 x 55 mm

Commit message: More Arranging
Parts:
- C24, R27, R28, R29, R30, R31, R37: moved to B.Cu
- R13, R23, R36, R49: footprint Resistor_SMD:R_0603_1608Metric_Pad0.98x0.95mm_HandSolder -> Resistor_SMD:R_0805_2012Metric_Pad1.20x1.40mm_HandSolder
- moved C9 186.7 mm to (55.2, 26.8)
- moved C21 173.3 mm to (244.3, 107.2), turned to -90 degrees
- moved J7 168.4 mm to (227.0, 80.0), turned to 180 degrees
- moved C5 168.3 mm to (223.7, 26.9)
- moved C24 166.5 mm to (241.9, 92.6), turned to 180 degrees
- moved U10 147.9 mm to (168.1, 96.9)
- moved U4 147.9 mm to (168.2, 103.5)
- moved R53 140.9 mm to (229.6, 114.7), turned to -90 degrees
- moved Q12 140.1 mm to (178.6, 114.2)
- moved J5 136.7 mm to (187.2, 126.8)
- moved U8 136.0 mm to (184.2, 86.8)
- moved J4 134.1 mm to (174.7, 126.9)
- moved TH1 132.3 mm to (227.6, 43.6)
- moved Q16 128.5 mm to (153.0, 161.1)
- moved D21 123.4 mm to (231.0, 112.0)
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- renumbered J7 to J5, J5 to J7
Connections:
- U10 pad 2: Net-(D15-A) -> /INFET3
- U10 pad 4: /INFET3 -> Net-(D15-A)
- U10 pad 5: +18V_DCIN -> /BAT3
- U10 pad 6: +18V_DCIN -> /BAT3
- U10 pad 7: /BAT3 -> +18V_DCIN
- U10 pad 8: /BAT3 -> +18V_DCIN
- U11 pad 2: Net-(D20-A) -> /INFET4
- U11 pad 4: /INFET4 -> Net-(D20-A)
- U11 pad 5: +18V_DCIN -> /BAT4
- U11 pad 6: +18V_DCIN -> /BAT4
- U11 pad 7: /BAT4 -> +18V_DCIN
- U11 pad 8: /BAT4 -> +18V_DCIN
Routing:
- net /BAT3: track 0.00 -> 20.0 mm, vias 0 -> 2
- net Net-(J17-DAT3/CD): track 0.00 -> 16.4 mm, vias 0 -> 2
- net GND: track 3.07 -> 17.0 mm, vias 3 -> 19
- net /SD_CS: track 0.00 -> 13.8 mm
- net /MISO: track 6.73 -> 19.4 mm, vias 0 -> 1
- net /SCK: track 13.4 -> 25.6 mm
- net Net-(J17-CLK): track 0.00 -> 8.58 mm
- net Net-(J17-CMD): track 0.00 -> 8.43 mm, vias 0 -> 2
- net Net-(U4-V_{CELL}): track 0.00 -> 8.00 mm
- net /MOSI: track 4.26 -> 11.5 mm
- net /VTEMP3: track 0.00 -> 5.94 mm, vias 0 -> 2
- net +5V: track 1.84 -> 7.14 mm, vias 0 -> 3
- net Net-(D13-K): track 0.00 -> 4.91 mm
- net Net-(D15-A): track 0.00 -> 4.89 mm
- net Net-(U4-SENSE): track 0.00 -> 4.84 mm
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- added copper zone on In2.Cu, net +3V3
- added copper zone on In2.Cu, net +5V

Commit message: MOSFETs changed
Parts:
- removed Q16, Q8: IRLZ44N, Package_TO_SOT_SMD:TO-252-2
- removed Q5, Q6, Q7: FQP27P06, Package_TO_SOT_SMD:TO-252-2
- added Q11: DMN3067LW-7, Package_TO_SOT_SMD:SOT-323_SC-70, F.Cu at (146.0, 160.3)
- added U12: Si4909DY-T1-GE3, Package_SO:SOIC-8_3.9x4.9mm_P1.27mm, F.Cu at (256.5, 29.6)
- added U13: Si4909DY-T1-GE3, Package_SO:SOIC-8_3.9x4.9mm_P1.27mm, F.Cu at (30.9, 25.3)
- D10, D5: footprint Diode_SMD:D_SMA_Handsoldering -> Diode_SMD:D_SOD-123F
- L1, L2, L3, L4: value 10u -> 10uH; footprint Inductor_SMD:L_0603_1608Metric_Pad1.05x0.95mm_HandSolder -> WE-LHMI_7050:WE-LHMI_7050
- Q1, Q3: value FQP27P06 -> DMP4065S-13; footprint Package_TO_SOT_SMD:TO-252-2 -> Package_TO_SOT_SMD:SOT-23
- Q12: value IRLZ44N -> DMN3067LW-7; footprint Package_TO_SOT_SMD:TO-252-2 -> Package_TO_SOT_SMD:SOT-323_SC-70
- Q2: value FQP27P06 -> 2N7002K; footprint Package_TO_SOT_SMD:TO-252-2 -> Package_TO_SOT_SMD:SOT-23
- Q4: value IRLZ44N -> 2N7002K; footprint Package_TO_SOT_SMD:TO-252-2 -> Package_TO_SOT_SMD:SOT-23
- TH1, TH2, TH3, TH4: footprint Resistor_SMD:R_0603_1608Metric_Pad0.98x0.95mm_HandSolder -> Connector_PinHeader_2.54mm:PinHeader_1x02_P2.54mm_Vertical
- moved Q4 221.2 mm to (43.3, 40.6)
- moved Q1 217.9 mm to (46.7, 32.2)
- moved L1 170.1 mm to (245.6, 50.7)
- moved D5 128.7 mm to (233.5, 22.7)
- moved TH4 93.3 mm to (124.9, 169.8)
- moved D10 89.0 mm to (26.4, 46.9)
- moved L4 83.4 mm to (129.3, 145.2)
- moved U7 66.3 mm to (201.0, 88.2)
- moved TH2 60.7 mm to (62.9, 26.2)
- moved U8 49.9 mm to (134.4, 88.5)
- moved L2 42.1 mm to (57.0, 38.2)
- moved TH3 29.1 mm to (183.9, 99.3), turned to 180 degrees
- moved R38 22.9 mm to (181.9, 103.7), turned to 0 degrees
- moved R37 22.9 mm to (181.8, 102.0), turned to 0 degrees
- moved C12 22.7 mm to (181.1, 99.3), turned to 90 degrees
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Connections:
- Q1 pad 1: /INFET1 -> /TGATE2
- Q1 pad 2: +34V_DCIN -> +34V_VCC
- Q1 pad 3: +34V_VCC -> /L2
- Q12 pad 2: /L3 -> GND
- Q12 pad 3: GND -> /L3
- Q2 pad 1: Net-(D5-A) -> /BGATE1
- Q2 pad 2: /BAT1 -> GND
- Q2 pad 3: +34V_VCC -> /L1
- Q3 pad 2: /L1 -> +34V_VCC
- Q3 pad 3: +34V_VCC -> /L1
- Q4 pad 1: /BGATE1 -> /BGATE2
- Q4 pad 2: /L1 -> GND
- Q4 pad 3: GND -> /L2
Routing:
- net Net-(U4-SENSE): track 4.84 -> 13.5 mm
- net /L3: track 0.00 -> 7.38 mm
- net /BGATE3: track 0.00 -> 5.78 mm
- net Net-(R37-Pad2): track 4.07 -> 7.35 mm
- net GND: vias 19 -> 20
Other:
- board size 125 x 55 mm -> 150 x 55 mm

Commit message: Board Done
Parts:
- added J8: Screw_Terminal_01x02, TerminalBlock_Phoenix:TerminalBlock_Phoenix_MKDS-1-2-3.81_1x02_P3.81mm_Horizontal, F.Cu at (129.1, 80.5)
- added J9: Screw_Terminal_01x02, TerminalBlock_Phoenix:TerminalBlock_Phoenix_MKDS-1-2-3.81_1x02_P3.81mm_Horizontal, F.Cu at (188.7, 80.5)
- C24, R27, R28, R29, R30, R31, R37: moved to F.Cu
- moved Q3 170.0 mm to (103.5, 105.9), turned to 180 degrees
- moved Q2 163.8 mm to (103.5, 102.3), turned to 180 degrees
- moved U12 163.6 mm to (113.5, 108.9)
- moved R17 158.2 mm to (153.8, 106.9), turned to 180 degrees
- moved R18 157.6 mm to (149.2, 115.0), turned to 180 degrees
- moved D5 153.2 mm to (108.3, 111.0), turned to -90 degrees
- moved U1 151.6 mm to (113.5, 102.5), turned to 180 degrees
- moved R3 150.3 mm to (122.7, 111.9), turned to 180 degrees
- moved C7 150.0 mm to (151.5, 99.4), turned to 90 degrees
- moved R1 149.7 mm to (119.1, 99.9)
- moved R2 147.7 mm to (119.1, 98.3)
- moved C8 147.7 mm to (148.9, 101.9)
- moved L1 146.8 mm to (105.8, 95.3), turned to 90 degrees
- moved R20 146.6 mm to (148.9, 100.3)
- moved R7 146.5 mm to (111.5, 112.5)
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Routing:
- net /SDA: track 0.00 -> 118.0 mm, vias 0 -> 4
- net /SCL: track 0.00 -> 114.7 mm, vias 0 -> 4
- net GND: track 17.0 -> 60.8 mm, vias 20 -> 47
- net /BAT2: track 0.00 -> 37.7 mm, vias 0 -> 2
- net /BAT1: track 0.00 -> 36.8 mm, vias 0 -> 2
- net /BAT4: track 0.00 -> 36.4 mm, vias 0 -> 2
- net +34V_VCC: track 0.00 -> 34.1 mm, vias 0 -> 7
- net +18V_VCC: track 0.00 -> 30.8 mm, vias 0 -> 7
- net Net-(D2-K): track 0.00 -> 23.6 mm, vias 0 -> 2
- net Net-(D17-K): track 0.00 -> 22.8 mm, vias 0 -> 2
- net Net-(D7-K): track 0.00 -> 21.9 mm, vias 0 -> 2
- net +34V_DCIN: track 0.00 -> 19.9 mm, vias 0 -> 10
- net +18V_DCIN: track 0.00 -> 17.7 mm, vias 1 -> 11
- net /BAT3: track 20.0 -> 37.5 mm
- net Net-(D12-K): track 4.03 -> 20.6 mm, vias 0 -> 2
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- added copper zone on In2.Cu, net +18V_DCIN
- added copper zone on In2.Cu, net +18V_VCC
- added copper zone on In2.Cu, net +34V_DCIN
- added copper zone on In2.Cu, net +34V_VCC

Commit message: Finishing Touches
Parts:
- removed J2: Screw_Terminal_01x02, TerminalBlock_Phoenix:TerminalBlock_Phoenix_MKDS-1-2-3.81_1x02_P3.81mm_Horizontal
- added C25: 10uF, Capacitor_THT:CP_Axial_L10.0mm_D4.5mm_P15.00mm_Horizontal, F.Cu at (120.0, 126.4)
- added J10: Barrel_Jack_MountingPin, Connector_BarrelJack:BarrelJack_GCT_DCJ200-10-A_Horizontal, F.Cu at (110.5, 124.5)
